File: MotionSimPCB/controllers.kicad_sch (KiCad schematic)
At the start: 18 parts, among them J11 Raspberry_Pi_4, U1 MPU-6050, U2 Teensy4.0

Commit message: fix drc, add protection
Parts:
- removed TP1, TP2, TP3, TP4: TestPoint, TestPoint:TestPoint_THTPad_D1.5mm_Drill0.7mm, symbol Connector:TestPoint
- added J13, J14: Conn_01x03, Connector_PinHeader_2.54mm:PinHeader_1x03_P2.54mm_Vertical, symbol Connector_Generic:Conn_01x03
- added R12, R7: 4.7k, Resistor_SMD:R_0805_2012Metric, symbol Device:R
- D3, D4, D5: JLC PN (none) -> C2289
- R10, R11, R8: value 10k -> 1k
Connections:
- net +3.3V: now also R12.1, R7.1
- net GND: now also U1.9 (AD0), J13.1 (Pin_1), J14.1 (Pin_1)
- net PI_RX: now also J13.2 (Pin_2)
- net PI_TX: now also J13.3 (Pin_3)
- net SCL: now also J14.2 (Pin_2), R12.2
- net SDA: now also J14.3 (Pin_3), R7.2

Commit message: fix clearance
Parts:
- C4: now in the parts list
- U1: footprint Sensor_Motion:InvenSense_QFN-24_3x3mm_P0.4mm -> Sensor_Motion:InvenSense_QFN-24_4x4mm_P0.5mm
Changed lines of the file:
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@@
 			)
 		)
-		(property "Footprint" "Sensor_Motion:InvenSense_QFN-24_3x3mm_P0.4mm"
+		(property "Footprint" "Sensor_Motion:InvenSense_QFN-24_4x4mm_P0.5mm"
 			(at 68.58 69.85 0)
 			(effects
@@
 		(unit 1)
 		(exclude_from_sim no)
-		(in_bom no)
+		(in_bom yes)
 		(on_board yes)
 		(dnp no)
